Commit message: falta arreglar TF urdf

File: src/teropobot_full/urdf/teropobot_full.urdf (robot description, URDF)
Before this commit: robot teropobot_full, 7 links, 6 joints
Joints:
- joint r_j1: limit lower=0 upper=0 effort=0 velocity=0 -> lower=-0.2 upper=0.11 effort=100 velocity=10; type continuous -> revolute
- joint r_j2: limit lower=0 upper=0 effort=0 velocity=0 -> lower=-1.57 upper=1.57 effort=100 velocity=10; type continuous -> revolute
- joint r_j3: limit lower=0 upper=0 effort=0 velocity=0 -> lower=-1.57 upper=0.2 effort=100 velocity=10; type continuous -> revolute
- joint r_j4: limit lower=0 upper=0 effort=0 velocity=0 -> lower=-1.57 upper=0.64 effort=100 velocity=10; type continuous -> revolute
- joint r_j5: limit lower=0 upper=0 effort=0 velocity=0 -> lower=-0.5 upper=1 effort=100 velocity=10; type continuous -> revolute
- joint s_j0: limit lower=0.1 upper=-0.1 effort=0 velocity=0 -> lower=-0.1 upper=0.1 effort=10 velocity=10

Commit message: TF arregladas

File: src/teropobot_full/urdf/teropobot_full.urdf (robot description, URDF)
Before this commit: robot teropobot_full, 7 links, 6 joints
Joints:
- joint r_j1: origin xyz=0.078905 -0.064 0.14462 rpy=0 0 0 -> xyz=0.078905 -0.064 0.13862 rpy=0 0 0
- joint r_j2: origin xyz=-0.022 -0.028 -0.069 rpy=0 0 0 -> xyz=-0.018 -0.028 -0.033 rpy=0 0 0

Commit message: Agrega l_leg

File: src/teropobot_full/urdf/teropobot_full.urdf (robot description, URDF)
Before this commit: robot teropobot_full, 7 links, 6 joints
Links:
- added link l_1, mass 0.247997823174623; collision mesh filename=package://teropobot_full/meshes/l_1.stl; visual mesh filename=package://teropobot_full/meshes/l_1.stl
- added link l_2, mass 0.0422410024350713; collision mesh filename=package://teropobot_full/meshes/l_2.stl; visual mesh filename=package://teropobot_full/meshes/l_2.stl
- added link l_3, mass 0.419694987008977; collision mesh filename=package://teropobot_full/meshes/l_3.stl; visual mesh filename=package://teropobot_full/meshes/l_3.stl
- added link l_4, mass 0.21645345011941; collision mesh filename=package://teropobot_full/meshes/l_4.stl; visual mesh filename=package://teropobot_full/meshes/l_4.stl
- added link l_5, mass 0.0778843023583795; collision mesh filename=package://teropobot_full/meshes/l_5.stl; visual mesh filename=package://teropobot_full/meshes/l_5.stl
Joints:
- added joint l_j1: type revolute, parent base_link, child l_1, origin xyz=0.078905 0.056 0.13862 rpy=0 0 0, axis 1 0 0, limit lower=-0.11 upper=0.2 effort=100 velocity=10
- added joint l_j2: type revolute, parent l_1, child l_2, origin xyz=-0.018 -0.028 -0.033 rpy=0 0 0, axis 0 1 0, limit lower=-1.57 upper=1.57 effort=100 velocity=10
- added joint l_j3: type revolute, parent l_2, child l_3, origin xyz=0 0 -0.125 rpy=0 0 0, axis 0 1 0, limit lower=-1.57 upper=0.2 effort=100 velocity=10
- added joint l_j4: type revolute, parent l_3, child l_4, origin xyz=0 0 -0.119 rpy=0 0 0, axis 0 1 0, limit lower=-1.57 upper=0.64 effort=100 velocity=10
- added joint l_j5: type revolute, parent l_4, child l_5, origin xyz=0 0 -0.0888 rpy=0 0 0, axis 0 1 0, limit lower=-0.5 upper=1 effort=100 velocity=10

Commit message: add head to s_0 link

File: src/teropobot_full/urdf/teropobot_full.urdf (robot description, URDF)
Before this commit: robot teropobot_full, 12 links, 11 joints
Links:
- link s_0: geometry collision mesh filename=package://teropobot_full/meshes/s_0_v4.stl; visual mesh filename=package://teropobot_full/meshes/s_0_v4.stl
Joints:
- joint l_j3: limit lower=-1.57 upper=0.2 effort=100 velocity=10 -> lower=-0.2 upper=1.57 effort=100 velocity=10
- joint r_j3: limit lower=-1.57 upper=0.2 effort=100 velocity=10 -> lower=-0.2 upper=1.57 effort=100 velocity=10
- joint s_j0: origin xyz=0.1634 0.0195 0.118455 rpy=0 0 0 -> xyz=0.1634 0.0195 0.122 rpy=0 0 0

Commit message: fix s_0 limits

File: src/teropobot_full/urdf/teropobot_full.urdf (robot description, URDF)
Before this commit: robot teropobot_full, 12 links, 11 joints
Joints:
- joint s_j0: limit lower=-0.1 upper=0.1 effort=10 velocity=10 -> lower=-0.06 upper=0.02 effort=10 velocity=10

Commit message: fix s_0

File: src/teropobot_full/urdf/teropobot_full.urdf (robot description, URDF)
Before this commit: robot teropobot_full, 12 links, 11 joints
Links:
- link s_0: geometry collision mesh filename=package://teropobot_full/meshes/s_0.stl; visual mesh filename=package://teropobot_full/meshes/s_0.stl

Commit message: rename links and joints

File: src/teropobot_full/urdf/teropobot_full.urdf (robot description, URDF)
Before this commit: robot teropobot_full, 12 links, 11 joints
Links:
- removed link l_1
- removed link l_2
- removed link l_3
- removed link l_4
- removed link l_5
- removed link r_1
- removed link r_2
- removed link r_3
- removed link r_4
- removed link r_5
- removed link s_0
- added link head_link, mass 0.187634452845745; collision mesh filename=package://teropobot_full/meshes/s_0.stl; visual mesh filename=package://teropobot_full/meshes/s_0.stl
- added link l_femur_link, mass 0.0422410024350713; collision mesh filename=package://teropobot_full/meshes/l_2.stl; visual mesh filename=package://teropobot_full/meshes/l_2.stl
- added link l_hip_link, mass 0.247997823174623; collision mesh filename=package://teropobot_full/meshes/l_1.stl; visual mesh filename=package://teropobot_full/meshes/l_1.stl
- added link l_metatarsals_link, mass 0.21645345011941; collision mesh filename=package://teropobot_full/meshes/l_4.stl; visual mesh filename=package://teropobot_full/meshes/l_4.stl
- added link l_phalanges_link, mass 0.0778843023583795; collision mesh filename=package://teropobot_full/meshes/l_5.stl; visual mesh filename=package://teropobot_full/meshes/l_5.stl
- added link l_tibia_link, mass 0.419694987008977; collision mesh filename=package://teropobot_full/meshes/l_3.stl; visual mesh filename=package://teropobot_full/meshes/l_3.stl
- added link r_femur_link, mass 0.0422410024350713; collision mesh filename=package://teropobot_full/meshes/r_2.stl; visual mesh filename=package://teropobot_full/meshes/r_2.stl
- added link r_hip_link, mass 0.247997823174623; collision mesh filename=package://teropobot_full/meshes/r_1.stl; visual mesh filename=package://teropobot_full/meshes/r_1.stl
- added link r_metatarsals_link, mass 0.21645345011941; collision mesh filename=package://teropobot_full/meshes/r_4.stl; visual mesh filename=package://teropobot_full/meshes/r_4.stl
- added link r_phalanges_link, mass 0.0778843023583795; collision mesh filename=package://teropobot_full/meshes/r_5.stl; visual mesh filename=package://teropobot_full/meshes/r_5.stl
- added link r_tibia_link, mass 0.419694987008977; collision mesh filename=package://teropobot_full/meshes/r_3.stl; visual mesh filename=package://teropobot_full/meshes/r_3.stl
Joints:
- removed joint l_j1
- removed joint l_j2
- removed joint l_j3
- removed joint l_j4
- removed joint l_j5
- removed joint r_j1
- removed joint r_j2
- removed joint r_j3
- removed joint r_j4
- removed joint r_j5
- removed joint s_j0
- added joint h_bobbing_joint: type prismatic, parent base_link, child head_link, origin xyz=0.1634 0.0195 0.122 rpy=0 0 0, axis 1 0 0, limit lower=-0.06 upper=0.02 effort=10 velocity=10
- added joint l_ankle_joint: type revolute, parent l_tibia_link, child l_metatarsals_link, origin xyz=0 0 -0.119 rpy=0 0 0, axis 0 1 0, limit lower=-1.57 upper=0.64 effort=100 velocity=10
- added joint l_hip_pitch_joint: type revolute, parent base_link, child l_hip_link, origin xyz=0.078905 0.056 0.13862 rpy=0 0 0, axis 1 0 0, limit lower=-0.11 upper=0.2 effort=100 velocity=10
- added joint l_hip_roll_joint: type revolute, parent l_hip_link, child l_femur_link, origin xyz=-0.018 -0.028 -0.033 rpy=0 0 0, axis 0 1 0, limit lower=-1.57 upper=1.57 effort=100 velocity=10
- added joint l_knee_joint: type revolute, parent l_femur_link, child l_tibia_link, origin xyz=0 0 -0.125 rpy=0 0 0, axis 0 1 0, limit lower=-0.2 upper=1.57 effort=100 velocity=10
- added joint l_phalanges_joint: type revolute, parent l_metatarsals_link, child l_phalanges_link, origin xyz=0 0 -0.0888 rpy=0 0 0, axis 0 1 0, limit lower=-0.5 upper=1 effort=100 velocity=10
- added joint r_ankle_joint: type revolute, parent r_tibia_link, child r_metatarsals_link, origin xyz=0 0 -0.119 rpy=0 0 0, axis 0 1 0, limit lower=-1.57 upper=0.64 effort=100 velocity=10
- added joint r_hip_pitch_joint: type revolute, parent base_link, child r_hip_link, origin xyz=0.078905 -0.064 0.13862 rpy=0 0 0, axis 1 0 0, limit lower=-0.2 upper=0.11 effort=100 velocity=10
- added joint r_hip_roll_joint: type revolute, parent r_hip_link, child r_femur_link, origin xyz=-0.018 -0.028 -0.033 rpy=0 0 0, axis 0 1 0, limit lower=-1.57 upper=1.57 effort=100 velocity=10
- added joint r_knee_joint: type revolute, parent r_femur_link, child r_tibia_link, origin xyz=0 0 -0.125 rpy=0 0 0, axis 0 1 0, limit lower=-0.2 upper=1.57 effort=100 velocity=10
- added joint r_phalanges_joint: type revolute, parent r_metatarsals_link, child r_phalanges_link, origin xyz=0 0 -0.0888 rpy=0 0 0, axis 0 1 0, limit lower=-0.5 upper=1 effort=100 velocity=10
